File: robot-motherboard/robot-motherboard.kicad_sch (KiCad schematic)
At the start: 0 parts

Commit message: Finish layout
Parts:
- added C1, C10, C11, C12, C2, C3, C6, C7, C8, C9: 100nF, Capacitor_THT:C_Disc_D3.0mm_W2.0mm_P2.50mm, symbol GS_Capacitor_THT:C_THT_Ceramic_Disk
- added C4, C5: 47uF, Capacitor_THT:CP_Radial_D5.0mm_P2.00mm, symbol GS_Capacitor_THT:C_THT_Electrolytic_Radial
- added G1: SSD1306_OLED, GS_Development_Boards:ADAFRUIT_SSD1306_OLED, symbol GS_Development_Boards:SSD1306_Breakout
- added H1, H2, H3, H4: M3_PTH, MountingHole:MountingHole_3.2mm_M3_Pad, symbol Mechanical:MountingHole_Pad
- added J1: Wing0_S, Connector_JST:JST_XH_B3B-XH-A_1x03_P2.50mm_Vertical, symbol Connector:Conn_01x03_Socket
- added J10: Reflectance, Connector_JST:JST_XH_B4B-XH-A_1x04_P2.50mm_Vertical, symbol Connector:Conn_01x04_Socket
- added J11: Arm_I, Connector_JST:JST_XH_B3B-XH-A_1x03_P2.50mm_Vertical, symbol Connector:Conn_01x03_Socket
- added J12: Intake_I, Connector_JST:JST_XH_B3B-XH-A_1x03_P2.50mm_Vertical, symbol Connector:Conn_01x03_Socket
- added J13: User.Input, TerminalBlock:TerminalBlock_Xinya_XY308-2.54-4P_1x04_P2.54mm_Horizontal, symbol Connector:Screw_Terminal_01x04
- added J14: I2C0, Connector_JST:JST_XH_B4B-XH-A_1x04_P2.50mm_Vertical, symbol Connector:Conn_01x04_Socket
- added J15: Extra, TerminalBlock:TerminalBlock_Xinya_XY308-2.54-5P_1x05_P2.54mm_Horizontal, symbol Connector:Screw_Terminal_01x05
- added J16: I2C1, Connector_JST:JST_XH_B4B-XH-A_1x04_P2.50mm_Vertical, symbol Connector:Conn_01x04_Socket
- added J2: Wing0_SW, Connector_JST:JST_XH_B3B-XH-A_1x03_P2.50mm_Vertical, symbol Connector:Conn_01x03_Socket
- added J3: BATT, Connector_JST:JST_XH_B2B-XH-A_1x02_P2.50mm_Vertical, symbol Connector:Conn_01x02_Socket
- added J4: Wing1_S, Connector_JST:JST_XH_B3B-XH-A_1x03_P2.50mm_Vertical, symbol Connector:Conn_01x03_Socket
- added J5: Wing1_SW, Connector_JST:JST_XH_B3B-XH-A_1x03_P2.50mm_Vertical, symbol Connector:Conn_01x03_Socket
- added J6: 9V, TerminalBlock:TerminalBlock_Xinya_XY308-2.54-2P_1x02_P2.54mm_Horizontal, symbol GS_Connectors:Screw_Terminal_01x02_2.54mm_Xinya
- added J7: Drivetrain_M, Connector_JST:JST_XH_B6B-XH-A_1x06_P2.50mm_Vertical, symbol Connector:Conn_01x05_Socket
- added J8, J9: Arm_M, Connector_JST:JST_XH_B6B-XH-A_1x06_P2.50mm_Vertical, symbol Connector:Conn_01x05_Socket
- added Q1: IRFZ44, Package_TO_SOT_THT:TO-220-3_Vertical, symbol GS_Transistors:MOSFET_N-Ch_60V_48A_23mR
- added R1: 470R, Resistor_THT:R_Axial_DIN0309_L9.0mm_D3.2mm_P12.70mm_Horizontal, symbol GS_Resistor_THT:R_250mW
- added R2: 10K, Resistor_THT:R_Axial_DIN0309_L9.0mm_D3.2mm_P12.70mm_Horizontal, symbol GS_Resistor_THT:R_250mW
- added R3, R4, R5, R6: 4k7, Resistor_THT:R_Axial_DIN0309_L9.0mm_D3.2mm_P12.70mm_Horizontal, symbol GS_Resistor_THT:R_250mW
- added RV1, RV2, RV3, RV4: POT0, GS_Resistors:ENPH253_Potentiometer, symbol Device:R_Potentiometer_US
- added S1: Logo, GS_Virtual:ENPH253_Logo, symbol GS_Virtual:ENPH253_Logo
- added U1: MCT6, Package_DIP:DIP-8_W7.62mm_LongPads, symbol GS_Optoelectronic:MCT6
- added U2: LM2596_Breakout, GS_Development_Boards:LM2596_Breakout, symbol GS_PMIC:LM2596_Breakout
- added U3: CD4051B, Package_DIP:DIP-16_W7.62mm_LongPads, symbol Analog_Switch:CD4051B
- added U4: ESP32_PICO-1, GS_Development_Boards:ESP32_PICO_1_DEV_KIT, symbol GS_Development_Boards:ESP32-PICO-KIT-1
- added U5: BNO085, GS_Development_Boards:ADAFRUIT_BNO085, symbol GS_IMU:ADAFRUIT_BNO085
Connections:
- new net: Q1.1 (G), R2.1, U1.7
- new net: RV2.2, U3.14 (X1)
- new net: J13.1 (Pin_1), U3.4 (X7)
- new net: J13.2 (Pin_2), U3.2 (X6)
- new net: J13.3 (Pin_3), U3.5 (X5)
- new net: J13.4 (Pin_4), U3.1 (X4)
- new net: C10.1, H2.1
- new net: RV1.2, U3.13 (X0)
- new net: C11.1, H3.1
- new net: RV4.2, U3.12 (X3)
- new net: RV3.2, U3.15 (X2)
- new net: R1.1, U1.1
- new net: C12.1, H4.1
- new net: C9.1, H1.1
- new net: Q1.2 (D), U2.4 (VOUT+)
- new net +3V3: C1.1, C2.1, C3.1, C4.1, C7.1, C8.1, G1.2 (VCC), J10.4 (Pin_4), J11.3 (Pin_3), J12.3 (Pin_3), J14.4 (Pin_4), J16.4 (Pin_4), R3.1, R4.1, R5.1, R6.1, RV1.1, RV2.1, RV3.1, RV4.1, U3.16 (VDD), U4.3V3, U5.1 (VIN), U5.9 (~{RST})
- new net +5V: C5.1, C6.1, Q1.3 (S), U4.5V
- new net +9V: J6.2 (Pin_2), R2.2, U2.1 (VIN+)
- new net +BATT: J3.2 (Pin_2), R1.2
- new net -BATT: J3.1 (Pin_1), U1.2
- new net ARM.INTAKE_DIR: J8.2 (Pin_2), J9.2 (Pin_2), U4.37 (GPIO37)
- new net ARM.INTAKE_PWM: J8.3 (Pin_3), J9.3 (Pin_3), U4.19 (GPIO19)
- new net ARM.INTAKE_SW: J12.2 (Pin_2), U4.20 (GPIO20)
- new net ARM.POSITION: J11.2 (Pin_2), U4.38 (GPIO38)
- new net ARM.SHOULDER_DIR: J8.4 (Pin_4), J9.4 (Pin_4), U4.9 (GPIO9)
- new net ARM.SHOULDER_PWM: J8.5 (Pin_5), J9.5 (Pin_5), U4.10 (GPIO10)
- new net DRIVETRAIN.M0_DIR: J7.4 (Pin_4), U4.14 (GPIO14)
- new net DRIVETRAIN.M0_PWM: J7.5 (Pin_5), U4.27 (GPIO27)
- new net DRIVETRAIN.M1_DIR: J7.2 (Pin_2), U4.4 (GPIO4)
- new net DRIVETRAIN.M1_PWM: J7.3 (Pin_3), U4.13 (GPIO13)
- new net GND: C1.2, C10.2, C11.2, C12.2, C2.2, C3.2, C4.2, C5.2, C6.2, C7.2, C8.2, C9.2, G1.1 (GND), J1.1 (Pin_1), J10.1 (Pin_1), J11.1 (Pin_1), J12.1 (Pin_1), J14.1 (Pin_1), J16.1 (Pin_1), J2.1 (Pin_1), J4.1 (Pin_1), J5.1 (Pin_1), J7.1 (Pin_1), J8.1 (Pin_1), J9.1 (Pin_1), RV1.3, RV2.3, RV3.3, RV4.3, U1.8, U2.3 (VOUT-), U3.6 (INH), U3.7 (VEE), U3.8 (VSS), U4.GND, U5.3 (GND)
- new net GNDPWR: J6.1 (Pin_1), U2.2 (VIN-)
- new net GPIO12: J15.1 (Pin_1), U4.12 (GPIO12)
- new net GPIO15: J15.2 (Pin_2), U4.15 (GPIO15)
- new net GPIO2: J15.3 (Pin_3), U4.2 (GPIO2)
- new net I2C0.SCL: G1.4 (SDA), J14.2 (Pin_2), R4.2, U4.22 (GPIO22), U5.5 (SDA)
- new net I2C0.SDA: G1.3 (SCL), J14.3 (Pin_3), R3.2, U4.21 (GPIO21), U5.4 (SCL)
- new net I2C1.SCL: J16.2 (Pin_2), R6.2, U4.5 (GPIO5)
- new net I2C1.SDA: J16.3 (Pin_3), R5.2, U4.0 (GPIO0)
- new net INPUT.MCU_IN: U3.3 (X), U4.26 (GPIO26)
- new net INPUT.SELECT0: U3.11 (A), U4.VP (GPIO36)
- new net INPUT.SELECT1: U3.10 (B), U4.VN (GPIO39)
- new net INPUT.SELECT2: U3.9 (C), U4.25 (GPIO25)
- new net IR0.IN: J10.3 (Pin_3), U4.34 (GPIO34)
- new net IR1.IN: J10.2 (Pin_2), U4.35 (GPIO35)
- new net RX0: J15.4 (Pin_4), U4.3 (RX0)
- new net TX0: J15.5 (Pin_5), U4.1 (TX0)
- new net WING0.LIMIT_SW_IN: J2.2 (Pin_2), U4.32 (GPIO32)
- new net WING0.SERVO: J1.2 (Pin_2), U4.8 (GPIO8)
- new net WING1.LIMIT_SW_IN: J5.2 (Pin_2), U4.33 (GPIO33)
- new net WING1.SERVO: J4.2 (Pin_2), U4.7 (GPIO7)
- no-connect marks 0 -> 16
Other:
- note added: "GPIO12 = MTDI GPIO15 = MTDO"
- note added: "MAKE SURE TO TEST STRAPPING BEFORE ORDERING!!!"
- note added: "Optional pull ups"

Commit message: Finish layout
Parts:
- added C13: 100nF, Capacitor_THT:C_Disc_D3.0mm_W2.0mm_P2.50mm, symbol GS_Capacitor_THT:C_THT_Ceramic_Disk
- added H5: M3_PTH, MountingHole:MountingHole_3.2mm_M3_Pad, symbol Mechanical:MountingHole_Pad
- added J17: PW_OUT, TerminalBlock:TerminalBlock_Xinya_XY308-2.54-3P_1x03_P2.54mm_Horizontal, symbol Connector:Screw_Terminal_01x03
- added J19: Basket_S, Connector_JST:JST_XH_B3B-XH-A_1x03_P2.50mm_Vertical, symbol Connector:Conn_01x03_Socket
- added JP1: Battery bypass, Jumper:SolderJumper-2_P1.3mm_Open_TrianglePad1.0x1.5mm, symbol Jumper:SolderJumper_2_Open
- J1, J2, J4, J5: footprint Connector_JST:JST_XH_B3B-XH-A_1x03_P2.50mm_Vertical -> GS_Connectors:JST_XH_S3B-XH-A-1_1x03_P2.50mm_Horizontal
- J14, J16: footprint Connector_JST:JST_XH_B4B-XH-A_1x04_P2.50mm_Vertical -> GS_Connectors:JST_XH_S4B-XH-A-1_1x04_P2.50mm_Horizontal
- J3: footprint Connector_JST:JST_XH_B2B-XH-A_1x02_P2.50mm_Vertical -> GS_Connectors:JST_XH_S2B-XH-A-1_1x02_P2.50mm_Horizontal
- J7, J8, J9: footprint Connector_JST:JST_XH_B6B-XH-A_1x06_P2.50mm_Vertical -> Connector_JST:JST_XH_B5B-XH-A_1x05_P2.50mm_Vertical
- Q1: footprint Package_TO_SOT_THT:TO-220-3_Vertical -> Package_TO_SOT_THT:TO-220-3_Horizontal_TabDown
- RV1: value POT0 -> POT1
- RV2: value POT0 -> POT2
- RV3: value POT0 -> POT3
- RV4: value POT0 -> POT4
Connections:
- net +3V3: now also RV1.3, RV2.3, RV3.3, RV4.3, J17.2 (Pin_2); no longer RV1.1, RV2.1, RV3.1, RV4.1
- net +5V: now also J17.3 (Pin_3), JP1.2 (B)
- net ARM.INTAKE_DIR: now also U4.9 (GPIO9); no longer U4.37 (GPIO37)
- net ARM.INTAKE_PWM: now also U4.10 (GPIO10); no longer U4.19 (GPIO19)
- net ARM.INTAKE_SW: now also U4.38 (GPIO38); no longer U4.20 (GPIO20)
- net ARM.POSITION: now also U4.37 (GPIO37); no longer U4.38 (GPIO38)
- net ARM.SHOULDER_DIR: now also U4.8 (GPIO8); no longer U4.9 (GPIO9)
- net ARM.SHOULDER_PWM: now also U4.19 (GPIO19); no longer U4.10 (GPIO10)
- net DRIVETRAIN.M0_DIR: now also U4.13 (GPIO13); no longer U4.14 (GPIO14)
- net DRIVETRAIN.M0_PWM: now also U4.4 (GPIO4); no longer U4.27 (GPIO27)
- net DRIVETRAIN.M1_DIR: now also U4.27 (GPIO27); no longer U4.4 (GPIO4)
- net DRIVETRAIN.M1_PWM: now also U4.14 (GPIO14); no longer U4.13 (GPIO13)
- net GND: now also J15.1 (Pin_1), RV1.1, RV2.1, RV3.1, RV4.1, C13.2, J17.1 (Pin_1), J19.1 (Pin_1); no longer RV1.3, RV2.3, RV3.3, RV4.3
- net GPIO12: now also J15.2 (Pin_2); no longer J15.1 (Pin_1)
- net IR0.IN: now also U4.35 (GPIO35); no longer U4.34 (GPIO34)
- net IR1.IN: now also U4.34 (GPIO34); no longer U4.35 (GPIO35)
- net WING0.SERVO: now also U4.7 (GPIO7); no longer U4.8 (GPIO8)
- net WING1.SERVO: now also U4.20 (GPIO20); no longer U4.7 (GPIO7)
- net at J13.1 (Pin_1): now also U3.1 (X4); no longer U3.4 (X7)
- net at J13.3 (Pin_3): now also U3.4 (X7); no longer U3.5 (X5)
- net at J13.4 (Pin_4): now also U3.5 (X5); no longer U3.1 (X4)
- net at Q1.2 (D), U2.4 (VOUT+): now also JP1.1 (A)
- net GPIO15 renamed BASKET.SERVO
- net BASKET.SERVO: now also J19.2 (Pin_2); no longer J15.2 (Pin_2)
- new net: C13.1, H5.1
- no-connect marks 16 -> 17
Other:
- moved on the sheet: C10, C11, C12, C2, C3, C4, C5, C6, C9, H1, H2, H3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

Commit message: Add filtering on user input
Parts:
- added C14, C15, C16, C17: 100nF, Capacitor_THT:C_Disc_D3.0mm_W2.0mm_P2.50mm, symbol GS_Capacitor_THT:C_THT_Ceramic_Disk
- RV1: value POT1 -> IN0
- RV2: value POT2 -> IN1
- RV3: value POT3 -> IN2
- RV4: value POT4 -> IN3
Connections:
- net +3V3: now also J1.3 (Pin_3), J19.3 (Pin_3), J2.3 (Pin_3), J4.3 (Pin_3), J5.3 (Pin_3)
- net GND: now also C14.2, C15.2, C16.2, C17.2
- net at RV2.2, U3.14 (X1): now also C15.1
- net at RV1.2, U3.13 (X0): now also C14.1
- net at RV4.2, U3.12 (X3): now also C17.1
- net at RV3.2, U3.15 (X2): now also C16.1
- no-connect marks 17 -> 12
Other:
- moved on the sheet: J1, J5, RV1, RV2, RV3, RV4, U1B

Commit message: Add switches between user input and encoder inputs
Parts:
- added J18: Encoder1, Connector_JST:JST_XH_B4B-XH-A_1x04_P2.50mm_Vertical, symbol Connector:Conn_01x04_Socket
- added J20: Encoder0, Connector_JST:JST_XH_B4B-XH-A_1x04_P2.50mm_Vertical, symbol Connector:Conn_01x04_Socket
- added SW1: ENC0.A/IN.SEL0, Button_Switch_THT:SW_Slide-03_Wuerth-WS-SLTV_10x2.5x6.4_P2.54mm, symbol Switch:SW_Wuerth_450301014042
- added SW2: ENC0.B/IN.SEL1, Button_Switch_THT:SW_Slide-03_Wuerth-WS-SLTV_10x2.5x6.4_P2.54mm, symbol Switch:SW_Wuerth_450301014042
- added SW3: ENC1.A/IN.SEL2, Button_Switch_THT:SW_Slide-03_Wuerth-WS-SLTV_10x2.5x6.4_P2.54mm, symbol Switch:SW_Wuerth_450301014042
- added SW4: ENC1.B/IN.ADC, Button_Switch_THT:SW_Slide-03_Wuerth-WS-SLTV_10x2.5x6.4_P2.54mm, symbol Switch:SW_Wuerth_450301014042
Connections:
- net +3V3: now also J18.4 (Pin_4), J20.4 (Pin_4)
- net GND: now also J18.1 (Pin_1), J20.1 (Pin_1)
- net INPUT.SELECT0: now also SW1.3 (A); no longer U4.VP (GPIO36)
- net INPUT.SELECT1: now also SW2.3 (A); no longer U4.VN (GPIO39)
- net INPUT.SELECT2: now also SW3.3 (A); no longer U4.25 (GPIO25)
- net INPUT.MCU_IN renamed INPUT.ADC_IN
- net INPUT.ADC_IN: now also SW4.3 (A); no longer U4.26 (GPIO26)
- new net ENCODER0.A: J20.3 (Pin_3), SW1.2 (C)
- new net ENCODER0.B: J20.2 (Pin_2), SW2.2 (C)
- new net ENCODER1.A: J18.3 (Pin_3), SW3.2 (C)
- new net ENCODER1.B: J18.2 (Pin_2), SW4.2 (C)
- new net SWITCH1: SW1.1 (B), U4.VP (GPIO36)
- new net SWITCH2: SW2.1 (B), U4.VN (GPIO39)
- new net SWITCH3: SW3.1 (B), U4.25 (GPIO25)
- new net SWITCH4: SW4.1 (B), U4.26 (GPIO26)
Other:
- moved on the sheet: C2, C3, C4, C5, C6, J10, J14, J16, R3, R4, R5, R6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

Commit message: Update to the right ESP32 footprint
Changed lines of the file:
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@@
 	(wire
 		(pts
-			(xy 302.26 198.12) (xy 276.86 198.12)
+			(xy 276.86 198.12) (xy 302.26 198.12)
 		)
 		(stroke
@@
 	(wire
 		(pts
-			(xy 302.26 218.44) (xy 276.86 218.44)
-		)
-		(stroke
-			(width 0)
-			(type default)
-		)
-	)
-	(wire
-		(pts
-			(xy 302.26 205.74) (xy 276.86 205.74)
+			(xy 276.86 218.44) (xy 302.26 218.44)
+		)
+		(stroke
+			(width 0)
+			(type default)
+		)
+	)
+	(wire
+		(pts
+			(xy 276.86 205.74) (xy 302.26 205.74)
 		)
 		(stroke
@@
 	(wire
 		(pts
-			(xy 302.26 220.98) (xy 276.86 220.98)
+			(xy 276.86 220.98) (xy 302.26 220.98)
 		)
 		(stroke
@@
 	(wire
 		(pts
-			(xy 302.26 203.2) (xy 276.86 203.2)
+			(xy 276.86 203.2) (xy 302.26 203.2)
 		)
 		(stroke
@@
 	(wire
 		(pts
-			(xy 302.26 187.96) (xy 276.86 187.96)
+			(xy 276.86 187.96) (xy 302.26 187.96)
 		)
 		(stroke
@@
 	(wire
 		(pts
-			(xy 302.26 223.52) (xy 276.86 223.52)
+			(xy 276.86 223.52) (xy 302.26 223.52)
 		)
 		(stroke
@@
 	(wire
 		(pts
-			(xy 302.26 200.66) (xy 276.86 200.66)
+			(xy 276.86 200.66) (xy 302.26 200.66)
 		)
 		(stroke
@@
 	(wire
 		(pts
-			(xy 302.26 190.5) (xy 276.86 190.5)
+			(xy 276.86 190.5) (xy 302.26 190.5)
 		)
 		(stroke
@@
 	(wire
 		(pts
-			(xy 302.26 195.58) (xy 276.86 195.58)
+			(xy 276.86 195.58) (xy 302.26 195.58)
 		)
 		(stroke
@@
 	(wire
 		(pts
-			(xy 302.26 193.04) (xy 276.86 193.04)
-		)
-		(stroke
-			(width 0)
-			(type default)
-		)
-	)
-	(wire
-		(pts
-			(xy 302.26 208.28) (xy 276.86 208.28)
+			(xy 276.86 193.04) (xy 302.26 193.04)
+		)
+		(stroke
+			(width 0)
+			(type default)
+		)
+	)
+	(wire
+		(pts
+			(xy 276.86 208.28) (xy 302.26 208.28)
 		)
 		(stroke
@@
 	(wire
 		(pts
-			(xy 302.26 215.9) (xy 276.86 215.9)
-		)
-		(stroke
+			(xy 276.86 215.9) (xy 302.26 215.9)
+		)
+		(stroke
